File: hardware/cubevox.kicad_sch (KiCad schematic)
At the start: 150 parts, among them J101 J_IN NCJ6FA-H, J106 DC 9V, J108 OUT 6.35mm, J117 OLED SH1106, K101 G6K-2F-Y DC5, K102 G6K-2F-Y DC5, Q101 MMBT3904, SW101 ST-0-102 bat toggle, SW102 ST-0-102 bat toggle, SW103 ST-0-102 bat toggle, SW104 ST-0-102 bat toggle, SW105 ST-0-102 bat toggle, SW106 ST-0-102 bat toggle, SW107 ST-0-102 bat toggle, SW108 ST-0-102 bat toggle, U101 CD74HC4067, U103 AP63205WU-7, U104 OPA2197IDR, U105 OPA2197IDR, U106 OPA2197IDR

Commit message: feat(hardware): pots RK09D1130C2P, encoders EC11E to match
Owner wants the 25 mm pot shaft. C2P (C361173) shares Alps drawing No. 4 with the C1B; only the shaft length differs, so pads stay. Encoders move to EC11E15244B2 (C470754, switch) and EC11E15204A3 (C470710) with the 24.5 mm tip; Alps drawings give EC11E the same PCB layout as EC11N. 3D models are the Alps C1B/EC11N STEPs with the shaft lengthened 5 mm inside the D-flat (tools/model_*.py), measured tips 25.0 and 24.5. Schematic regenerated with every pin on its old net, ERC 0; board D0184 ledger 0225, DRC 0, netlist parity 0/0/0.
Parts:
- ENC101: value EC11N1525404 -> EC11E15244B2; footprint cubevox:SW-TH_EC11NXXXX -> cubevox:SW-TH_EC11E; symbol cubevox:EC11N1525404 -> cubevox:EC11E15244B2; LCSC C470748 -> C470754; MPN EC11N1525404 -> EC11E15244B2
- ENC102, ENC103: value EC11N1520401 -> EC11E15204A3; footprint cubevox:SW-TH_EC11NXXXX -> cubevox:SW-TH_EC11E; symbol cubevox:EC11N1520401 -> cubevox:EC11E15204A3; LCSC C470703 -> C470710; MPN EC11N1520401 -> EC11E15204A3
- RV101, RV102, RV103, RV104, RV105, RV106, RV107, RV108, RV109, RV110, RV111, RV112, RV113, RV114, RVGAIN1: footprint cubevox:RES-ADJ-TH_RK09D1130C3C -> cubevox:RES-ADJ-TH_RK09D1130C2P; symbol cubevox:RK09D1130C1B -> cubevox:RK09D1130C2P; LCSC C470304 -> C361173; MPN RK09D1130C1B -> RK09D1130C2P

Commit message: feat(hardware): reassign MCU pins to the edge facing each destination
The old map left 14 of 35 local nets on the U1 edge facing away from
their parts. Each movable net now leaves the facing edge in fan-out
order, I2C moves to I2C2 on the OLED corner, CC1/CC2 come off the MCU
(USB is data only) and MUTE_N avoids the JTAG pull-up pins. The
VA_SENSE divider moves beside U106's 5VA pin with its cap at the MCU.
Connections:
- net I2C1_SCL renamed I2C_SCL
- net I2C1_SDA renamed I2C_SDA
Other:
- sheet h7core_block ports: added I2C_SCL, I2C_SDA; removed I2C1_SCL, I2C1_SDA
Changed lines of the file:
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@@
 		)
 	)
-	(label "I2C1_SCL"
+	(label "I2C_SCL"
 		(at 791.21 598.17 180)
 		(fields_autoplaced yes)
@@
 		)
 	)
-	(label "I2C1_SDA"
+	(label "I2C_SDA"
 		(at 791.21 600.71 180)
 		(fields_autoplaced yes)
@@
 		)
 	)
-	(label "I2C1_SCL"
+	(label "I2C_SCL"
 		(at 848.36 603.25 270)
 		(fields_autoplaced yes)
@@
 		)
 	)
-	(label "I2C1_SDA"
+	(label "I2C_SDA"
 		(at 863.6 603.25 270)
 		(fields_autoplaced yes)
@@
 			)
 		)
-		(pin "I2C1_SCL" bidirectional
+		(pin "I2C_SCL" bidirectional
 			(at 83.82 105.41 0)
 			(effects
@@
 			)
 		)
-		(pin "I2C1_SDA" bidirectional
+		(pin "I2C_SDA" bidirectional
 			(at 83.82 109.22 0)
 			(effects
@@
 		)
 	)
-	(label "I2C1_SCL"
+	(label "I2C_SCL"
 		(at 86.36 105.41 0)
 		(fields_autoplaced yes)
@@
 		)
 	)
-	(label "I2C1_SDA"
+	(label "I2C_SDA"
 		(at 86.36 109.22 0)
 		(fields_autoplaced yes)
