File: hardware/cubevox.kicad_sch (KiCad schematic)
At the start: 163 parts, among them J101 J_IN NCJ6FA-H, J106 DC 9V, J108 OUT 6.35mm, J117 OLED SH1106, K102 G6K-2F-Y DC5, K103 G6K-2F-Y DC5, Q101 MMBT3904, Q102 MMBT3904, SW101 ST-0-102 bat toggle, SW102 ST-0-102 bat toggle, SW103 ST-0-102 bat toggle, SW104 ST-0-102 bat toggle, SW105 ST-0-102 bat toggle, SW106 ST-0-102 bat toggle, SW107 ST-0-102 bat toggle, SW108 ST-0-102 bat toggle, U101 CD74HC4067, U103 AP63205WU-7, U104 OPA2197IDR, U105 OPA2197IDR, U106 OPA2197IDR, U108 OPA197IDBVR

Commit message: fix(hardware): pre-fab audit fixes, pad relay on NC contacts, MUX_S0 pull-down
Five read-only audits (fab limits, assembly, electrical, ground return,
renders) against c2635eb; reports under docs/audits/2026-10-10-prefab-*.md.

K103 had IN_P and LINE_N on the NO contacts, so coil off left the 25.7 dB
pad in circuit; c4788e2 wants coil off = MIC. IN_P moves to pin 2 and
LINE_N to pin 7 (NC); IN_N stays on COM pin 6; the board is re-laid with
a B.Cu lane between the relay pad rows. C127 now feeds U105.8 on F.Cu in
the 5VA chain. The GND via inside D2.2 goes. R162 100k pulls MUX_S0 low:
PE12 is the ROM bootloader's SPI4 SCK while PE11 holds its NSS, and a
floating clock could lock the bootloader off USB DFU. RESET/BOOT silk at
0.15 mm. Project hole-to-hole rule 0.50 mm. PARTS.md, PINMAP, the spec
and pins.h carry PAD_EN on PE11 and the new parts; make_bom.py writes
CPL rotations 0 to 359.

gates.sh ALL PASS (DRC 9 lib mismatches, 0 unconnected, parity clean),
mega_audit loops 0 jogs 7 acute 0 nearmiss 0 edgebend 0, ERC 0.
Parts:
- added R162: 100k, Resistor_SMD:R_0402_1005Metric, symbol Device:R
Connections:
- net GND: now also R162.2
- net IN_P: now also K103.2; no longer K103.4
- net LINE_N: now also K103.7; no longer K103.5
- net MUX_S0: now also R162.1
Changed lines of the file:
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@@
 	)
 	(no_connect
-		(at 970.28 581.66)
+		(at 985.52 581.66)
 	)
 	(wire
@@
 	(wire
 		(pts
-			(xy 985.52 581.66) (xy 985.52 594.36)
+			(xy 970.28 581.66) (xy 970.28 594.36)
 		)
 		(stroke
@@
 	)
 	(label "IN_P"
-		(at 985.52 594.36 270)
+		(at 970.28 594.36 270)
 		(fields_autoplaced yes)
 		(effects
@@
 	(wire
 		(pts
-			(xy 985.52 562.61) (xy 985.52 549.91)
+			(xy 970.28 562.61) (xy 970.28 549.91)
 		)
 		(stroke
@@
 	)
 	(label "LINE_N"
-		(at 985.52 549.91 90)
+		(at 970.28 549.91 90)
 		(fields_autoplaced yes)
 		(effects
@@
 	)
 	(no_connect
-		(at 970.28 562.61)
+		(at 985.52 562.61)
 	)
 	(wire
@@
 		(fields_autoplaced yes)
 		(effects
+			(font
+				(size 1.27 1.27)
+			)
+			(justify right bottom)
+		)
+	)
+	(symbol
+		(lib_id "Device:R")
+		(at 111.76 115.57 0)
+		(unit 1)
+		(exclude_from_sim no)
+		(in_bom yes)
+		(on_board yes)
+		(dnp no)
+		(property "Reference" "R162"
+			(at 114.3 114.3 0)
+			(effects
+				(font
+					(size 1.27 1.27)
+				)
+				(justify left)
+			)
+		)
+		(property "Value" "100k"
+			(at 114.3 116.84 0)
+			(effects
+				(font
+					(size 1.27 1.27)
+				)
+				(justify left)
+			)
+		)
+		(property "Footprint" "Resistor_SMD:R_0402_1005Metric"
+			(at 111.76 115.57 0)
+			(hide yes)
+			(effects
+				(font
+					(size 1.27 1.27)
+				)
+			)
+		)
+		(property "Datasheet" "~"
+			(at 111.76 115.57 0)
+			(hide yes)
+			(effects
+				(font
+					(size 1.27 1.27)
+				)
+			)
+		)
+		(property "LCSC" "C25741"
+			(at 111.76 115.57 0)
+			(hide yes)
+			(effects
+				(font
+					(size 1.27 1.27)
+				)
+			)
+		)
+		(pin "1"
+		)
+		(pin "2"
+		)
+		(instances
+			(project "cubevox"
+				(path "/99ad1494-2bf8-5051-8886-2c8b83c86254"
+					(reference "R162")
+					(unit 1)
+				)
+			)
+		)
+	)
+	(wire
+		(pts
+			(xy 111.76 109.22) (xy 111.76 111.76)
+		)
+		(stroke
+			(width 0)
+			(type default)
+		)
+	)
+	(wire
+		(pts
+			(xy 111.76 119.38) (xy 111.76 121.92)
+		)
+		(stroke
+			(width 0)
+			(type default)
+		)
+	)
+	(label "MUX_S0"
+		(at 111.76 109.22 90)
+		(fields_autoplaced yes)
+		(effects
+			(font
+				(size 1.27 1.27)
+			)
+			(justify left bottom)
+		)
+	)
+	(label "GND"
+		(at 111.76 121.92 270)
+		(fields_autoplaced yes)
+		(effects

Commit message: fix(hardware): JLC footprints for U107, U108, C19; production v4
The H7 core block came from a KiCad-library project, so U107 (SOT-23),
U108 (SOT-23-5) and C19 (EIA-6032 tantalum) kept stock footprints whose
zero orientation is 180 degrees from JLC's. The v3 CPL therefore had all
three turned round. Each now uses the easyeda2kicad footprint for its
LCSC number (C412495, C221351, C8649) at the same centre; the track
ends, TP10, the U107 ground via and the C19 5 V via follow the 0.13 to
0.30 mm pad shifts. Every assembled asymmetric part is now on a JLC
footprint. gates.sh ALL PASS, mega_audit loops 0, ERC 0.

Production v4: BOM 73 lines / 223 parts, CPL 223 rows, U107 90, U108
180, C19 180 degrees. v2 and v3 are superseded; upload v4 only.
Parts:
- U108: footprint Package_TO_SOT_SMD:SOT-23-5 -> cubevox_h7core:SOT-23-5_L3.0-W1.7-P0.95-LS2.8-BR
Changed lines of the file:
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@@
 			)
 		)
-		(property "Footprint" "Package_TO_SOT_SMD:SOT-23-5"
+		(property "Footprint" "cubevox_h7core:SOT-23-5_L3.0-W1.7-P0.95-LS2.8-BR"
 			(at 619.76 455.93 0)
 			(effects
